File: modsimple.sch (KiCad schematic (older format))
At the start: 9 parts, among them J1 MICROUSB, P1 CONN_10, Q2 FDD8870, U1 MAX1811

Commit message: moved to MCP73831
Parts:
- removed U1: MAX1811, symbol MAX1811
- added R?: 2K, symbol R
- added U?: MCP73831, ~, symbol MCP73831
- C1, C2: value 10uF -> 4.7uF
Connections:
- wire segments 55 -> 46
Other:
- note removed: "Vsel: High = 4.2V Low = 4.1V\nIsel: High = 500mA Low = 100mA"
- moved on the sheet: C1, C2, R1, R3
Changed lines of the file:
@@
-EESchema Schematic File Version 2  date Mon 25 Mar 2013 10:46:17 AM CDT
+EESchema Schematic File Version 2  date Tue 26 Mar 2013 10:51:40 AM CDT
 LIBS:power
 LIBS:device
@@
 Sheet 1 1
 Title ""
-Date "24 mar 2013"
+Date "26 mar 2013"
 Rev ""
 Comp ""
@@
 L R R3
 U 1 1 5133879A
-P 7350 4550
-F 0 "R3" V 7430 4550 50  0000 C CNN
-F 1 "330" V 7350 4550 50  0000 C CNN
-F 2 "" H 7350 4550 60  0001 C CNN
-F 3 "" H 7350 4550 60  0001 C CNN
-	1    7350 4550
+P 7550 4400
+F 0 "R3" V 7630 4400 50  0000 C CNN
+F 1 "330" V 7550 4400 50  0000 C CNN
+F 2 "" H 7550 4400 60  0001 C CNN
+F 3 "" H 7550 4400 60  0001 C CNN
+	1    7550 4400
 	-1   0    0    1
 $EndComp
@@
 L GND #PWR2
 U 1 1 512B9659
-P 6450 4750
-F 0 "#PWR2" H 6450 4750 30  0001 C CNN
-F 1 "GND" H 6450 4680 30  0001 C CNN
-F 2 "" H 6450 4750 60  0001 C CNN
-F 3 "" H 6450 4750 60  0001 C CNN
-	1    6450 4750
+P 4750 4750
+F 0 "#PWR2" H 4750 4750 30  0001 C CNN
+F 1 "GND" H 4750 4680 30  0001 C CNN
+F 2 "" H 4750 4750 60  0001 C CNN
+F 3 "" H 4750 4750 60  0001 C CNN
+	1    4750 4750
 	1    0    0    -1
 $EndComp
@@
 L C C2
 U 1 1 512B964A
-P 6450 4500
-F 0 "C2" H 6500 4600 50  0000 L CNN
-F 1 "10uF" H 6500 4400 50  0000 L CNN
-F 2 "" H 6450 4500 60  0001 C CNN
-F 3 "" H 6450 4500 60  0001 C CNN
-	1    6450 4500
+P 4750 4350
+F 0 "C2" H 4800 4450 50  0000 L CNN
+F 1 "4.7uF" H 4800 4250 50  0000 L CNN
+F 2 "" H 4750 4350 60  0001 C CNN
+F 3 "" H 4750 4350 60  0001 C CNN
+	1    4750 4350
 	1    0    0    -1
 $EndComp
@@
 L GND #PWR1
 U 1 1 512B9625
-P 3850 3850
-F 0 "#PWR1" H 3850 3850 30  0001 C CNN
-F 1 "GND" H 3850 3780 30  0001 C CNN
-F 2 "" H 3850 3850 60  0001 C CNN
-F 3 "" H 3850 3850 60  0001 C CNN
-	1    3850 3850
+P 7000 3300
+F 0 "#PWR1" H 7000 3300 30  0001 C CNN
+F 1 "GND" H 7000 3230 30  0001 C CNN
+F 2 "" H 7000 3300 60  0001 C CNN
+F 3 "" H 7000 3300 60  0001 C CNN
+	1    7000 3300
 	1    0    0    -1
 $EndComp
@@
 L C C1
 U 1 1 512B9601
-P 4100 3950
-F 0 "C1" H 4150 4050 50  0000 L CNN
-F 1 "10uF" H 4150 3850 50  0000 L CNN
-F 2 "" H 4100 3950 60  0001 C CNN
-F 3 "" H 4100 3950 60  0001 C CNN
-	1    4100 3950
-	1    0    0    -1
+P 6800 3400
+F 0 "C1" H 6850 3500 50  0000 L CNN
+F 1 "4.7uF" H 6850 3300 50  0000 L CNN
+F 2 "" H 6800 3400 60  0001 C CNN
+F 3 "" H 6800 3400 60  0001 C CNN
+	1    6800 3400
+	-1   0    0    1
 $EndComp
 $Comp
 L R R1
 U 1 1 512B94C6
-P 3950 4950
-F 0 "R1" V 4030 4950 50  0000 C CNN
-F 1 "330" V 3950 4950 50  0000 C CNN
-F 2 "" H 3950 4950 60  0001 C CNN
-F 3 "" H 3950 4950 60  0001 C CNN
-	1    3950 4950
+P 3950 6100
+F 0 "R1" V 4030 6100 50  0000 C CNN
+F 1 "330" V 3950 6100 50  0000 C CNN
+F 2 "" H 3950 6100 60  0001 C CNN
+F 3 "" H 3950 6100 60  0001 C CNN
+	1    3950 6100
 	0    -1   -1   0
 $EndComp
@@
 Text Label 10050 3500 2    60   ~ 0
 FireLED-
-$Comp
-L MAX1811 U1
-U 1 1 514F4034
-P 5500 4350
-F 0 "U1" H 5500 5000 60  0000 C CNN
-F 1 "MAX1811" H 5500 4350 60  0000 C CNN
-F 2 "" H 5500 4350 60  0000 C CNN
-F 3 "" H 5500 4350 60  0000 C CNN
-	1    5500 4350
-	1    0    0    -1
-$EndComp
 Wire Wire Line
 	8450 3100 8450 3000
@@
 Wire Wire Line
 	10050 3100 8800 3100
-Connection ~ 7350 4250
-Wire Wire Line
-	7350 4250 7350 4300
-Wire Wire Line
-	7600 5100 8600 5100
-Wire Wire Line
-	8800 4250 6150 4250
-Wire Wire Line
-	8800 3100 8800 4250
+Wire Wire Line
+	7750 5100 8600 5100
+Wire Wire Line
+	8800 3100 8800 3950
 Wire Wire Line
 	3700 2600 11100 2600
@@
 	8900 5300 8900 5450
 Wire Wire Line
-	6450 4700 6450 4750
-Wire Wire Line
-	4100 4150 4100 4250
-Wire Wire Line
-	3700 4250 4850 4250
-Wire Wire Line
 	11100 2600 11100 3200
 Wire Wire Line
-	6450 4250 6450 4300
-Connection ~ 6450 4250
-Wire Wire Line
-	3700 2600 3700 4950
+	4750 3600 4750 4150
+Wire Wire Line
+	3700 2600 3700 6100
 Wire Wire Line
 	11100 3600 11200 3600
@@
 Connection ~ 8800 3300
 Wire Wire Line
-	7350 4800 7550 4800
-Wire Wire Line
-	7550 4800 7550 6050
-Wire Wire Line
 	7550 6050 9050 6050
 Wire Wire Line
@@
 	9050 3600 10050 3600
 Wire Wire Line
-	4200 4950 7500 4950
-Wire Wire Line
-	7500 4950 7500 6100
-Wire Wire Line
-	7500 6100 9100 6100
+	4200 6100 9100 6100
 Wire Wire Line
 	9100 6100 9100 3700
@@
 	9500 3900 9500 4450
 Wire Wire Line
-	9500 4450 7600 4450
-Wire Wire Line
-	7600 4450 7600 5100
+	9500 4450 7750 4450
+Wire Wire Line
+	7750 4450 7750 5100
 Wire Wire Line
 	10050 3500 8900 3500
 Connection ~ 8900 3500
 Wire Wire Line
-	4450 3750 4450 4100
-Wire Wire Line
-	4450 4100 4850 4100
-Connection ~ 4100 4250
-Wire Wire Line
-	3850 3750 4450 3750
-Connection ~ 4100 3750
-Wire Wire Line
-	6150 4100 8750 4100
-Wire Wire Line
-	8750 4100 8750 3000
-Connection ~ 8750 3000
-Connection ~ 3700 4250
-Wire Wire Line
-	4650 3950 4850 3950
-Wire Wire Line
-	9200 6150 6800 6150
-Wire Wire Line
-	6800 6150 6800 3800
-Wire Wire Line
-	6800 3800 6150 3800
-Text Notes 4700 2950 0    60   ~ 0
-Vsel: High = 4.2V Low = 4.1V\nIsel: High = 500mA Low = 100mA
-Wire Wire Line
-	3850 3750 3850 3850
-Wire Wire Line
-	4850 3800 4650 3800
-Wire Wire Line
-	4650 3600 4650 4250
-Connection ~ 4650 4250
-Connection ~ 4650 3950
-Wire Wire Line
-	6150 3950 6400 3950
-Wire Wire Line
-	6400 3950 6400 3600
-Wire Wire Line
-	6400 3600 4650 3600
-Connection ~ 4650 3800
+	7000 3200 6800 3200
+Wire Wire Line
+	9200 6150 4400 6150
+Wire Wire Line
+	4400 6150 4400 3300
+Wire Wire Line
+	7000 3200 7000 3300
+$Comp
+L MCP73831 U?
+U 1 1 5151B767
+P 5400 3700
+F 0 "U?" H 5400 4200 60  0000 C CNN
+F 1 "MCP73831" H 5400 3700 60  0000 C CNN
+F 2 "~" H 5400 3700 60  0000 C CNN
+F 3 "~" H 5400 3700 60  0000 C CNN
+	1    5400 3700
+	1    0    0    -1
+$EndComp
+Wire Wire Line
+	6500 2600 6500 3600
+Wire Wire Line
+	6050 3600 6800 3600
+Connection ~ 6500 2600
+Connection ~ 6500 3600
+Wire Wire Line
+	4750 4550 4750 4750
+$Comp
+L GND #PWR?
+U 1 1 5151C31D
+P 4550 3550
+F 0 "#PWR?" H 4550 3550 30  0001 C CNN
+F 1 "GND" H 4550 3480 30  0001 C CNN
+F 2 "" H 4550 3550 60  0001 C CNN
+F 3 "" H 4550 3550 60  0001 C CNN
+	1    4550 3550
+	1    0    0    -1
+$EndComp
+Wire Wire Line
+	4750 3450 4550 3450
+Wire Wire Line
+	4550 3200 4550 3550
+Wire Wire Line
+	8800 3950 4750 3950
+Connection ~ 4750 3950
+Wire Wire Line
+	7550 4150 7550 3950
+Connection ~ 7550 3950
+Wire Wire Line
+	7550 4650 7550 6050
+Wire Wire Line
+	4400 3300 4750 3300
+$Comp
+L R R?
+U 1 1 5151C561
+P 4550 2950
+F 0 "R?" V 4630 2950 50  0000 C CNN
+F 1 "2K" V 4550 2950 50  0000 C CNN
+F 2 "" H 4550 2950 60  0001 C CNN
+F 3 "" H 4550 2950 60  0001 C CNN
+	1    4550 2950
+	-1   0    0    1
+$EndComp
+Wire Wire Line
+	6050 2700 6050 3300
+Connection ~ 4550 3450
+Wire Wire Line
+	6050 2700 4550 2700
 $EndSCHEMATC

Commit message: part selection changes (again)
Parts:
- gave numbers to parts that had none: 2
Changed lines of the file:
@@
-EESchema Schematic File Version 2  date Tue 26 Mar 2013 10:51:40 AM CDT
+EESchema Schematic File Version 2  date Wed 27 Mar 2013 01:11:27 AM CDT
 LIBS:power
 LIBS:device
@@
 $EndComp
 $Comp
-L GND #PWR3
+L GND #PWR4
 U 1 1 513187A3
 P 7950 5800
-F 0 "#PWR3" H 7950 5800 30  0001 C CNN
+F 0 "#PWR4" H 7950 5800 30  0001 C CNN
 F 1 "GND" H 7950 5730 30  0001 C CNN
 F 2 "" H 7950 5800 60  0001 C CNN
@@
 Atomizer-
 $Comp
-L GND #PWR5
+L GND #PWR6
 U 1 1 51302ACE
 P 8900 5450
-F 0 "#PWR5" H 8900 5450 30  0001 C CNN
+F 0 "#PWR6" H 8900 5450 30  0001 C CNN
 F 1 "GND" H 8900 5380 30  0001 C CNN
 F 2 "" H 8900 5450 60  0001 C CNN
@@
 Battery+
 $Comp
-L GND #PWR6
+L GND #PWR7
 U 1 1 512C4AF2
 P 11200 3800
-F 0 "#PWR6" H 11200 3800 30  0001 C CNN
+F 0 "#PWR7" H 11200 3800 30  0001 C CNN
 F 1 "GND" H 11200 3730 30  0001 C CNN
 F 2 "" H 11200 3800 60  0001 C CNN
@@
 $EndComp
 $Comp
-L GND #PWR1
+L GND #PWR3
 U 1 1 512B9625
 P 7000 3300
-F 0 "#PWR1" H 7000 3300 30  0001 C CNN
+F 0 "#PWR3" H 7000 3300 30  0001 C CNN
 F 1 "GND" H 7000 3230 30  0001 C CNN
 F 2 "" H 7000 3300 60  0001 C CNN
@@
 $EndComp
 $Comp
-L GND #PWR4
+L GND #PWR5
 U 1 1 512AF9E3
 P 8450 3100
-F 0 "#PWR4" H 8450 3100 30  0001 C CNN
+F 0 "#PWR5" H 8450 3100 30  0001 C CNN
 F 1 "GND" H 8450 3030 30  0001 C CNN
 F 2 "" H 8450 3100 60  0001 C CNN
@@
 	7000 3200 7000 3300
 $Comp
-L MCP73831 U?
+L MCP73831 U1
 U 1 1 5151B767
 P 5400 3700
-F 0 "U?" H 5400 4200 60  0000 C CNN
+F 0 "U1" H 5400 4200 60  0000 C CNN
 F 1 "MCP73831" H 5400 3700 60  0000 C CNN
 F 2 "~" H 5400 3700 60  0000 C CNN
@@
 	4750 4550 4750 4750
 $Comp
-L GND #PWR?
+L GND #PWR1
 U 1 1 5151C31D
 P 4550 3550
-F 0 "#PWR?" H 4550 3550 30  0001 C CNN
+F 0 "#PWR1" H 4550 3550 30  0001 C CNN
 F 1 "GND" H 4550 3480 30  0001 C CNN
 F 2 "" H 4550 3550 60  0001 C CNN
@@
 	4400 3300 4750 3300
 $Comp
-L R R?
+L R R4
 U 1 1 5151C561
 P 4550 2950
-F 0 "R?" V 4630 2950 50  0000 C CNN
+F 0 "R4" V 4630 2950 50  0000 C CNN
 F 1 "2K" V 4550 2950 50  0000 C CNN
 F 2 "" H 4550 2950 60  0001 C CNN

Commit message: morning updates
Connections:
- net Atomizer+ renamed Vbat
- net Atomizer- renamed Atty-
- net Switch- renamed GATE
Other:
- note added: "Connections to booster backpack:\nAtomizer+ to Vbat\nSwitch - to GATE\nFireLED- to Atty-\nBattery- to GND (tap from wires, NOT from PCB. Keep connected to board!)"
- note added: "NOTE! FireLED- Will not work as intended!\n(I.e. to light an LED when fire button is pressed.)\nHowever, no changes to be made because this pin is useful for the backpack\n"
Changed lines of the file:
@@
-EESchema Schematic File Version 2  date Wed 27 Mar 2013 01:11:27 AM CDT
+EESchema Schematic File Version 2  date Mon 01 Apr 2013 08:03:03 AM CDT
 LIBS:power
 LIBS:device
@@
 LIBS:valves
 LIBS:mod
-LIBS:modsimple-cache
+LIBS:mod-cache
 EELAYER 27 0
 EELAYER END
 $Descr A4 11693 8268
 encoding utf-8
-Sheet 1 1
+Sheet 3 3
 Title ""
-Date "26 mar 2013"
+Date "1 apr 2013"
 Rev ""
 Comp ""
@@
 $EndComp
 $Comp
-L GND #PWR4
+L GND #PWR05
 U 1 1 513187A3
 P 7950 5800
-F 0 "#PWR4" H 7950 5800 30  0001 C CNN
+F 0 "#PWR05" H 7950 5800 30  0001 C CNN
 F 1 "GND" H 7950 5730 30  0001 C CNN
 F 2 "" H 7950 5800 60  0001 C CNN
@@
 Atomizer-
 $Comp
-L GND #PWR6
+L GND #PWR06
 U 1 1 51302ACE
 P 8900 5450
-F 0 "#PWR6" H 8900 5450 30  0001 C CNN
+F 0 "#PWR06" H 8900 5450 30  0001 C CNN
 F 1 "GND" H 8900 5380 30  0001 C CNN
 F 2 "" H 8900 5450 60  0001 C CNN
@@
 Battery+
 $Comp
-L GND #PWR7
+L GND #PWR07
 U 1 1 512C4AF2
 P 11200 3800
-F 0 "#PWR7" H 11200 3800 30  0001 C CNN
+F 0 "#PWR07" H 11200 3800 30  0001 C CNN
 F 1 "GND" H 11200 3730 30  0001 C CNN
 F 2 "" H 11200 3800 60  0001 C CNN
@@
 $EndComp
 $Comp
-L GND #PWR2
+L GND #PWR08
 U 1 1 512B9659
 P 4750 4750
-F 0 "#PWR2" H 4750 4750 30  0001 C CNN
+F 0 "#PWR08" H 4750 4750 30  0001 C CNN
 F 1 "GND" H 4750 4680 30  0001 C CNN
 F 2 "" H 4750 4750 60  0001 C CNN
@@
 $EndComp
 $Comp
-L GND #PWR3
+L GND #PWR09
 U 1 1 512B9625
 P 7000 3300
-F 0 "#PWR3" H 7000 3300 30  0001 C CNN
+F 0 "#PWR09" H 7000 3300 30  0001 C CNN
 F 1 "GND" H 7000 3230 30  0001 C CNN
 F 2 "" H 7000 3300 60  0001 C CNN
@@
 $EndComp
 $Comp
-L GND #PWR5
+L GND #PWR010
 U 1 1 512AF9E3
 P 8450 3100
-F 0 "#PWR5" H 8450 3100 30  0001 C CNN
+F 0 "#PWR010" H 8450 3100 30  0001 C CNN
 F 1 "GND" H 8450 3030 30  0001 C CNN
 F 2 "" H 8450 3100 60  0001 C CNN
@@
 FireLED-
 Wire Wire Line
-	8450 3100 8450 3000
+	8450 2800 8450 3100
 Wire Wire Line
 	8450 3000 10050 3000
@@
 	7950 5700 7950 5800
 Wire Wire Line
-	8800 3200 10050 3200
+	8200 3200 10050 3200
 Connection ~ 8800 3200
 Connection ~ 8800 3300
@@
 	9500 3900 9500 4450
 Wire Wire Line
-	9500 4450 7750 4450
+	7750 4450 9750 4450
 Wire Wire Line
 	7750 4450 7750 5100
 Wire Wire Line
-	10050 3500 8900 3500
+	8050 3500 10050 3500
 Connection ~ 8900 3500
 Wire Wire Line
@@
 	4750 4550 4750 4750
 $Comp
-L GND #PWR1
+L GND #PWR011
 U 1 1 5151C31D
 P 4550 3550
-F 0 "#PWR1" H 4550 3550 30  0001 C CNN
+F 0 "#PWR011" H 4550 3550 30  0001 C CNN
 F 1 "GND" H 4550 3480 30  0001 C CNN
 F 2 "" H 4550 3550 60  0001 C CNN
@@
 Wire Wire Line
 	6050 2700 4550 2700
+Text HLabel 8050 3100 0    60   Output ~ 0
+Vbat
+Text Notes 9650 4150 0    60   ~ 0
+NOTE! FireLED- Will not work as intended!\n(I.e. to light an LED when fire button is pressed.)\nHowever, no changes to be made because this pin is useful for the backpack\n
+Text Notes 7850 1950 0    60   ~ 0
+Connections to booster backpack:\nAtomizer+ to Vbat\nSwitch - to GATE\nFireLED- to Atty-\nBattery- to GND (tap from wires, NOT from PCB. Keep connected to board!)
+Wire Wire Line
+	8050 3100 8200 3100
+Wire Wire Line
+	8200 3100 8200 3200
+Text HLabel 8050 2800 0    60   Input ~ 0
+GND
+Text HLabel 9750 4450 2    60   Input ~ 0
+GATE
+Connection ~ 9500 4450
+Wire Wire Line
+	8050 2800 8450 2800
+Connection ~ 8450 3000
+Text HLabel 8050 3500 0    60   Output ~ 0
+Atty-
 $EndSCHEMATC
