File: modsimple.sch (KiCad schematic (older format))
At the start: 10 parts, among them J1 MICROUSB, P1 CONN_10, Q2 FDD8870, U1 MCP73831

Commit message: Main sheet integration progress
Connections:
- net Vusb: now reaches C1.1, J1.1 (Vbus), R1.1, U1.4 (Vdd)
Changed lines of the file:
@@
-EESchema Schematic File Version 2  date Wed 03 Apr 2013 10:52:06 AM CDT
+EESchema Schematic File Version 2  date Thu 04 Apr 2013 10:55:40 AM CDT
 LIBS:power
 LIBS:device
@@
 Sheet 3 4
 Title ""
-Date "3 apr 2013"
+Date "4 apr 2013"
 Rev ""
 Comp ""
@@
 Text HLabel 8050 3500 0    60   Output ~ 0
 Atty-
+Text HLabel 11100 2600 2    60   Input ~ 0
+Vusb
 $EndSCHEMATC
