File: mod.sch (KiCad schematic (older format))
At the start: 16 parts, among them IC1 ATTINY85-S, J1 MICROUSB, P1 CONN_12, Q2 FDD8870, SW1 SW_PUSH_SMALL, SW2 SW_PUSH_SMALL, SW3 SW_PUSH_SMALL

Commit message: morning updates
Parts:
- removed J1: MICROUSB, symbol MICROUSB
- removed Q2: FDD8870, symbol MOSFET_N
- removed R2: 10K, symbol R
- removed R9: 330, symbol R
- P2: renamed from P1; symbol CONN_12 -> CONN_10
Connections:
- net ChargeLED+ is gone; now on net UP-MCU: P2.8 (P8)
- net ChargeLED- is gone; now on net DWN-MCU: P2.9 (P9)
- net Atomizer-: now also P2.4 (P4); no longer P2.5 (P5)
- net DWN-MCU: no longer P2.11 (P11)
- net FIRE-MCU: now also P2.10 (P10); no longer P2.12 (P12)
- net GND: no longer P2.4 (P4)
- net UP-MCU: no longer P2.10 (P10)
- net Simple PCB/GATE: now reaches IC1.5 (PB0(MOSI/DI/SDA/AIN0/OC0A/OC1A/AREF/PCINT0))
Other:
- note added: "Vdiv resistor values not yet set!"
- moved on the sheet: R10, R11, R12, R8
