File: Boost.sch (KiCad schematic (older format))
At the start: 19 parts, among them Q1 FDD8870, U2 LTC1871

Commit message: adsf
Changed lines of the file:
@@
-EESchema Schematic File Version 2  date Thu 04 Apr 2013 10:55:40 AM CDT
+EESchema Schematic File Version 2  date Fri 05 Apr 2013 11:43:57 PM CDT
 LIBS:power
 LIBS:device
@@
 Sheet 2 4
 Title ""
-Date "4 apr 2013"
+Date "5 apr 2013"
 Rev ""
 Comp ""
@@
 	6550 2550 7900 2550
 Connection ~ 7500 2550
+Text HLabel 2900 4300 2    60   Input ~ 0
+GND
 $EndSCHEMATC
