File: mod.kicad_pcb (KiCad board)
At the start: 2 copper layers, 44 parts, among them IC1 ATTINY85-S, J1 MICROUSB, P1 CONN_12, Q1 FDD8870, Q2 FDD8870, SW1 SW_PUSH_SMALL, SW2 SW_PUSH_SMALL, SW3 SW_PUSH_SMALL, U1 MCP73831, U2 LTC1871

Commit message: progress on layout
Parts:
- C1, C2, D1, D2, IC1, J1, Q2, R1, R10, R11, R12, R13, R2, R3, R4, R5, R6, R7, R8, R9, U1: moved to B.Cu
- D3: footprint TO263 -> DPAK2_Schottky
- moved SW3 145.2 mm to (0.00, 0.00)
- moved SW2 135.3 mm to (0.00, 0.00)
- moved SW1 126.2 mm to (0.00, 0.00)
- moved R6 61.1 mm to (101.7, 23.7), turned to 180 degrees
- moved R5 57.8 mm to (101.7, 25.8), turned to 180 degrees
- moved R7 49.4 mm to (101.7, 28.8), turned to 180 degrees
- moved R8 47.5 mm to (101.7, 30.9)
- moved R2 34.9 mm to (90.3, 27.6), turned to 0 degrees
- moved R13 34.6 mm to (78.6, 27.7), turned to 90 degrees
- moved IC1 33.4 mm to (96.8, 28.5), turned to 0 degrees
- moved Q2 32.8 mm to (90.4, 27.8), turned to 270 degrees
- moved C4 32.4 mm to (60.1, 77.6), turned to 90 degrees
- moved C2 32.3 mm to (76.7, 31.2), turned to 270 degrees
- moved R4 31.9 mm to (75.1, 24.6), turned to 180 degrees
- moved P1 31.4 mm to (83.9, 22.5)
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Connections:
- C10 pad 1: (no net) -> /Boost/Vout
- C10 pad 2: (no net) -> GND
- IC1 pad 3: N-000006 -> /UP-MCU
- IC1 pad 6: N-000005 -> N-000008
- IC1 pad 7: /UP-MCU -> N-000005
- Q2 pad G: N-000006 -> N-000004
- R2 pad 2: N-000006 -> N-000004
- R5 pad 2: /Atomizer- -> N-000008
- R6 pad 2: N-000005 -> N-000008
- R7 pad 2: N-000004 -> N-000005
- R8 pad 1: N-000004 -> N-000005
Routing:
- net N-0000019: track 0.00 -> 63.2 mm, vias 0 -> 3
- net /Boost/Vout: track 31.1 -> 90.8 mm
- net GND: track 0.00 -> 52.0 mm, vias 0 -> 6
- net /MCP73831 Charger/Vbat: track 27.8 -> 71.9 mm
- net /Atomizer-: track 0.00 -> 37.9 mm
- net /UP-MCU: track 0.00 -> 13.0 mm
- net N-000008: track 0.00 -> 12.8 mm
- net N-000004: track 0.00 -> 12.4 mm
- net /DWN-MCU: track 0.00 -> 11.1 mm
- net N-000005: track 0.00 -> 10.2 mm
- net /FIRE-MCU: track 0.00 -> 6.98 mm
- net N-0000024: track 0.00 -> 4.78 mm
- net N-0000023: track 8.26 -> 4.37 mm
- net N-0000027: track 0.00 -> 3.88 mm
- net /FireLED+: track 0.00 -> 2.04 mm
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- added copper zone on B.Cu, net /Atomizer-
- added copper zone on B.Cu, net /MCP73831 Charger/Vcharge
- added copper zone on B.Cu, net GND
- added copper zone on F.Cu, net GND
- added copper zone on B.Cu, net N-0000019
- added copper zone on F.Cu, net N-0000019

Commit message: many changes. Most not stable. Check TODO
Parts:
- removed the C2 at (76.7, 31.2)
- removed the J1 at (63.5, 26.7)
- removed SW1, SW2, SW3: SW_PUSH_SMALL, SW_PUSH_SMALL
- added C1: 4.7uF, SM0805, F.Cu at (140.3, 76.6)
- added C2: 4.7uF, SM0805, F.Cu at (75.7, 26.5)
- added C2: 4.7uF, SM0805, F.Cu at (141.5, 73.4)
- added J1: MICROUSB, USBmicro, F.Cu at (68.3, 29.3)
- added J1: MICROUSB, USBmicro, F.Cu at (132.0, 79.1)
- added P1: CONN_10, SIL-10, F.Cu at (139.0, 70.5)
- added Q2: FDD8870, TO-252_Mosfet, B.Cu at (147.7, 74.8)
- added R1: 330, SM0805, F.Cu at (128.3, 72.9)
- added R2: 10K, SM0805, B.Cu at (147.7, 74.8)
- added R3: 330, SM0805, F.Cu at (145.2, 73.4)
- added R4: 2K, SM0805, F.Cu at (146.2, 76.6)
- added U1: MCP73831, SOT23-5, F.Cu at (143.4, 76.3)
- C1, D1, D2, R1, R13, R4, U1: moved to F.Cu
- moved D1 16.6 mm to (86.4, 28.3), turned to 90 degrees
- moved Q2 14.0 mm to (76.3, 27.7), turned to 90 degrees
- moved R2 9.66 mm to (82.2, 32.9), turned to 270 degrees
- moved R4 7.78 mm to (79.9, 30.7), turned to 90 degrees
- moved D2 6.05 mm to (84.6, 30.4), turned to 270 degrees
- moved R6 4.62 mm to (97.3, 25.0)
- moved R5 4.59 mm to (97.3, 26.9)
- moved R7 4.45 mm to (97.3, 29.1)
- moved R8 4.45 mm to (97.3, 31.1)
- moved IC1 4.45 mm to (92.4, 28.8)
- moved U1 4.41 mm to (78.7, 27.1), turned to 180 degrees
- moved R13 4.24 mm to (82.8, 28.3), turned to 270 degrees
- moved C1 3.34 mm to (77.9, 30.7)
- moved R1 2.97 mm to (75.3, 30.2)
Connections:
- IC1 pad 1: /FIRE-MCU -> /UP-MCU
- IC1 pad 3: /UP-MCU -> /FIRE-MCU
Routing:
- net /chgLED+: track 0.00 -> 25.3 mm
- net /Atomizer+: track 0.00 -> 17.0 mm
- net /MCP73831 Charger/ChargeLED-: track 0.00 -> 15.5 mm
- net N-000004: track 12.4 -> 27.8 mm
- net N-000009: track 0.00 -> 14.0 mm
- net /Atomizer-: track 37.9 -> 48.1 mm
- net N-0000027: track 3.88 -> 11.8 mm
- net /chgLED-: track 0.00 -> 7.27 mm
- net /Switch-: track 0.00 -> 6.97 mm
- net /UP-MCU: track 13.0 -> 6.87 mm
- net /FireLED+: track 2.04 -> 6.74 mm
- net GND: track 52.0 -> 56.3 mm
- net /DWN-MCU: track 11.1 -> 8.09 mm
- net /FIRE-MCU: track 6.98 -> 9.07 mm
- net N-0000025: track 0.00 -> 1.79 mm
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- added copper zone on F.Cu, net /MCP73831 Charger/Vcharge
- removed copper zone on B.Cu, net /Atomizer-
- removed copper zone on B.Cu, net /MCP73831 Charger/Vcharge
Other:
- board outline added: 84.1 x 61.8 mm
- net class Default: clearance 0.2286 -> 0.254
- net class High Power removed
- net class Low Power: clearance 0.2286 -> 0.254
- net class Power added: clearance 0.127, trace_width 1.016, via_dia 0.889, via_drill 0.635
- rule trace_clearance: 0.2286 -> 0.254
- board text added: "Cled+"
- board text added: "Cled-"
- board text added: "DWN"
- board text added: "FIRE"
- board text added: "Fled+"
- board text added: "UP"
